Commit message: robot joints issue fixes

File: catkin_ws/src/my_robot/urdf/my_robot.xacro (robot description, xacro)
@@ -6,4 +6,6 @@
 <xacro:property name="wheel_length" value="0.05" />
 <xacro:property name="ground_gap_offset" value="0.1" />
+<xacro:property name="small_wheel_radius" value="0.05" />
+<xacro:property name="small_wheel_length" value="0.025" />
 <xacro:include filename="$(find my_robot)/urdf/my_robot.gazebo"/>
 <link name="robot_footprint"></link>
@@ -16,5 +18,5 @@
     <pose xyz="0 0 ${chassis_size_z}" rpy="0 0 0" />
     <inertial>
-    <mass value="15.0"/>
+    <mass value="10.0"/>
     <origin xyz="0 0 0" rpy="0 0 0"/>
     <inertia ixx="0.1" ixy="0" ixz="0"
@@ -35,6 +37,32 @@
         <material name="Orange"/>
         </visual>
-</link>
-<link name="chassis_extra">
+    </link>
+<link name='chassis_head'>
+    <pose xyz="0 0 0" rpy="0 0 0" />
+    <inertial>
+    <mass value="0.1"/>
+    <origin xyz="0 0 0" rpy="0 0 0"/>
+    <inertia ixx="0.1" ixy="0" ixz="0"
+            iyy="0.1" iyz="0"
+            izz="0.1"/>
+    </inertial>
+    <collision name='chassis_head_collision'>
+    <origin xyz="0 0 ${chassis_size_z + chassis_size_z/8}" rpy=" 0 0 0"/>
+        <geometry>
+        <sphere radius="${chassis_size_x/4}"/>
+        </geometry>
+    </collision>
+    <visual name='chassis_head_visual'>
+    <origin xyz="0 0 ${chassis_size_z + chassis_size_z/8}" rpy=" 0 0 0"/>
+        <geometry>
+        <sphere radius="${chassis_size_x/4}"/>
+        </geometry>
+    </visual>
+</link>
+<joint name="chassis_head_joint" type="fixed">
+<parent link="chassis"/>
+<child link="chassis_head"/>
+</joint>
+<link name="back_wheel_chassis">
     <pose xyz="0 0 ${chassis_size_z}" rpy="0 0 0" />
     <inertial>
@@ -45,112 +73,116 @@
             izz="0.1"/>
     </inertial>
-            <collision name='chassis_caster_stand_collision'>
-        <origin xyz="${-(chassis_size_x/2.0 - ground_gap_offset/2.0)} 0 ${-((chassis_size_z/2.0 - ground_gap_offset/2.0)/2.0)}" rpy=" 0 0 0"/>
-            <geometry>
-            <box size="${ground_gap_offset} ${ground_gap_offset} ${chassis_size_z/2.0 - ground_gap_offset/2}"/>
+    <collision name='back_wheel_chassis_collision'>
+    <origin xyz="${-(chassis_size_x/2.0 - ground_gap_offset/2.0)} 0 ${-((chassis_size_z/2.0 - ground_gap_offset/2.0)/2.0)}" rpy=" 0 0 0"/>
+        <geometry>
+        <box size="${ground_gap_offset} ${ground_gap_offset} ${chassis_size_z/2.0 - ground_gap_offset/2}"/>
+        </geometry>
+    </collision>
+    <visual name='back_wheel_chassis_visual'>
+    <origin xyz="${-(chassis_size_x/2.0 - ground_gap_offset/2.0)} 0  ${-((chassis_size_z/2.0 - ground_gap_offset/2.0)/2.0)}" rpy=" 0 0 0"/>
+        <geometry>
+        <box size="${ground_gap_offset} ${ground_gap_offset} ${chassis_size_z/2.0 - ground_gap_offset/2.0}"/>
+        </geometry>
+        <material name="brown"/>
+    </visual>
+</link>
+<joint name="back_wheel_chassis_joint" type="fixed">
+<parent link="chassis"/>
+<child link="back_wheel_chassis"/>
+</joint>
+<link name="back_chassis_wheel">
+    <pose xyz="0 0 0" rpy="0 0 0" />
+    <inertial>
+    <mass value="0.1"/>
+    <origin xyz="0 0 0" rpy="0 0 0"/>
+    <inertia ixx="0.1" ixy="0" ixz="0"
+            iyy="0.1" iyz="0"
+            izz="0.1"/>
+    </inertial>
+    <collision name='back_chassis_wheel_collision'>
+    <origin xyz="0 0 0" rpy="0 0 0"/>
+        <geometry>
+        <sphere radius="${ground_gap_offset/2.0}"/>
+        </geometry>
+    </collision>
+    <visual name='back_chassis_wheel_visual'>
+    <origin xyz="0 0 0" rpy="0 0 0"/>
+        <geometry>
+        <sphere radius="${ground_gap_offset/2.0}"/>
+        </geometry>
+        <material name = "back_chassis_wheel">
+            <color rgba="1 0 0 1"/>
+            </material>
+    </visual>
+</link>
+<joint name="back_chassis_caster_hinge" type="continuous">
+<origin xyz="${-(chassis_size_x/2.0 - ground_gap_offset/2.0)} 0  ${-((chassis_size_z/2.0- ground_gap_offset/2.0))}" rpy="0 0 0"/>
+<parent link="chassis"/>
+<child link="back_chassis_wheel"/>
+<axis xyz="0 1 0" rpy="0 0 0"/>
+<axis2 xyz="1 0 0" rpy="0 0 0"/>
+</joint>
+<link name="front_wheel_chassis">
+    <pose xyz="0 0 ${chassis_size_z}" rpy="0 0 0" />
+    <inertial>
+    <mass value="1.0"/>
+    <origin xyz="0 0 0" rpy="0 0 0"/>
+    <inertia ixx="0.1" ixy="0" ixz="0"
+            iyy="0.1" iyz="0"
+            izz="0.1"/>
+    </inertial>
+          <collision name='front_wheel_chassis_collision'>
+        <origin xyz="${(chassis_size_x/2.0 - ground_gap_offset/2.0)} 0  ${-((chassis_size_z/2.0 - ground_gap_offset/2.0)/2.0)}" rpy=" 0 0 0"/>
+            <geometry>
+            <box size="${ground_gap_offset} ${ground_gap_offset} ${chassis_size_z/2.0 - ground_gap_offset/2.0}"/>
             </geometry>
         </collision>
-        <visual name='chassis_caster_stand_visual'>
-        <origin xyz="${-(chassis_size_x/2.0 - ground_gap_offset/2.0)} 0  ${-((chassis_size_z/2.0 - ground_gap_offset/2.0)/2.0)}" rpy=" 0 0 0"/>
+        <visual name='front_wheel_chassis_visual'>
+        <origin xyz="${(chassis_size_x/2.0 - ground_gap_offset/2.0)} 0  ${-((chassis_size_z/2.0- ground_gap_offset/2.0)/2.0)}" rpy=" 0 0 0"/>
             <geometry>
             <box size="${ground_gap_offset} ${ground_gap_offset} ${chassis_size_z/2.0 - ground_gap_offset/2.0}"/>
             </geometry>
-         <material name="chassis_extra"/>
+          <material name="Gray"/>
         </visual>
-          <collision name='chassis_caster_stand_collision'>
-        <origin xyz="${(chassis_size_x/2.0 - ground_gap_offset/2.0)} 0  ${-((chassis_size_z/2.0 - ground_gap_offset/2.0)/2.0)}" rpy=" 0 0 0"/>
-            <geometry>
-            <box size="${ground_gap_offset} ${ground_gap_offset} ${chassis_size_z/2.0 - ground_gap_offset/2.0}"/>
-            </geometry>
-        </collision>
-        <visual name='chassis_caster_stand_visual'>
-        <origin xyz="${(chassis_size_x/2.0 - ground_gap_offset/2.0)} 0  ${-((chassis_size_z/2.0- ground_gap_offset/2.0)/2.0)}" rpy=" 0 0 0"/>
-            <geometry>
-            <box size="${ground_gap_offset} ${ground_gap_offset} ${chassis_size_z/2.0 - ground_gap_offset/2.0}"/>
-            </geometry>
-          <material name="chassis_extra"/>
-        </visual>
-        <collision name='chassis_head_collision'>
-        <origin xyz="0 0 ${chassis_size_z + chassis_size_z/8}" rpy=" 0 0 0"/>
-            <geometry>
-            <sphere radius="${chassis_size_x/4}"/>
-            </geometry>
-        </collision>
-        <visual name='chassis_head_visual'>
-        <origin xyz="0 0 ${chassis_size_z + chassis_size_z/8}" rpy=" 0 0 0"/>
-            <geometry>
-            <sphere radius="${chassis_size_x/4}"/>
-            </geometry>
-        <material name="chassis_extra"/>
-        </visual>
-</link>
-<joint name="chassis_extra_joint" type="fixed">
-<orgin xyz="0 0 0" rpy="0 0 0"/>
-<parent link="chassis"/>
-<child link="chassis_extra"/>
-</joint>
-<link name="back_chassis_caster">
-    <pose xyz="0 0 ${chassis_size_z}" rpy="0 0 0" />
-    <inertial>
-    <mass value="0.1"/>
-    <origin xyz="0 0 0" rpy="0 0 0"/>
-    <inertia ixx="0.1" ixy="0" ixz="0"
-            iyy="0.1" iyz="0"
-            izz="0.1"/>
-    </inertial>
-    <collision name='back_caster_collision'>
-    <origin xyz="${-(chassis_size_x/2.0 - ground_gap_offset/2.0)} 0 ${-chassis_size_z/2.0+ground_gap_offset/2.0}" rpy=" 0 0 0"/>
-        <geometry>
-        <sphere radius="${ground_gap_offset/2}"/>
-        </geometry>
-    </collision>
-    <visual name='back_caster_visual'>
-    <origin xyz="${-(chassis_size_x/2.0 - ground_gap_offset/2.0)} 0 ${-chassis_size_z/2.0+ground_gap_offset/2.0}" rpy=" 0 0 0"/>
+</link>
+<joint name="front_wheel_chassis_joint" type="fixed">
+<orgin xyz="${(chassis_size_x/2.0 - ground_gap_offset/2.0)} 0  ${-((chassis_size_z/2.0- ground_gap_offset/2.0)/2.0)}" rpy="0 0 0"/>
+<parent link="chassis"/>
+<child link="front_wheel_chassis"/>
+</joint>
+<link name="front_chassis_wheel">
+<pose xyz="0 0 0" rpy="0 0 0" />
+     <inertial>
+        <mass value="5.0"/>
+        <origin xyz="0 0 0" rpy="0 0 0"/>
+        <inertia ixx="0.1" ixy="0" ixz="0"
+                iyy="0.1" iyz="0"
+                izz="0.1"/>
+        </inertial>
+    <collision name='front_chassis_wheel_collision'>
+    <origin xyz="0 0 0" rpy="0 0 0"/>
         <geometry>
         <sphere radius="${ground_gap_offset/2.0}"/>
         </geometry>
-        <material name="Blue"/>
-    </visual>
-</link>
-<link name="front_chassis_caster">
-    <pose xyz="0 0 ${chassis_size_z}" rpy="0 0 0" />
-    <inertial>
-    <mass value="0.1"/>
-    <origin xyz="0 0 0" rpy="0 0 0"/>
-    <inertia ixx="0.1" ixy="0" ixz="0"
-            iyy="0.1" iyz="0"
-            izz="0.1"/>
-    </inertial>
-        <collision name='front_caster_collision'>
-        <origin xyz="${chassis_size_x/2.0 - ground_gap_offset/2.0} 0 ${-chassis_size_z/2.0+ground_gap_offset/2.0}" rpy=" 0 0 0"/>
-            <geometry>
-            <sphere radius="${ground_gap_offset/2.0}"/>
-            </geometry>
-        </collision>
-        <visual name='front_caster_visual'>
-        <origin xyz="${chassis_size_x/2.0 - ground_gap_offset/2.0} 0 ${-chassis_size_z/2.0+ground_gap_offset/2.0}" rpy=" 0 0 0"/>
-            <geometry>
-            <sphere radius="${ground_gap_offset/2.0}"/>
-            </geometry>
-            <material name="Blue"/>
-        </visual>
-</link>
-<joint type="revolute" name="back_caster_joint">
-<orgin xyz="0 0 0" rpy="0 0 0"/>
-<parent link="chassis"/>
-<child link="back_chassis_caster"/>
+    </collision>
+    <visual name='front_chassis_wheel_visual'>
+    <origin xyz="0 0 0" rpy="0 0 0"/>
+        <geometry>
+        <sphere radius="${ground_gap_offset/2.0}"/>
+        </geometry>
+        <material name = "front_chassis_wheel">
+            <color rgba="1 0 0 1"/>
+            </material>
+    </visual>
+</link>
+<joint name="front_chassis_caster_hinge" type="continuous">
+<origin xyz="${(chassis_size_x/2.0 - ground_gap_offset/2.0)} 0  ${-((chassis_size_z/2.0- ground_gap_offset/2.0))}" rpy="0 0 0"/>
+<parent link="chassis"/>
+<child link="front_chassis_wheel"/>
 <axis xyz="0 1 0" rpy="0 0 0"/>
 <axis2 xyz="1 0 0" rpy="0 0 0"/>
-<limit effort="1000.0" lower="0.0" upper="3.14" velocity="0.5"/>
-</joint>
-<joint name="front_caster_joint" type="revolute">
-<orgin xyz="${chassis_size_x/2.0 - ground_gap_offset/2.0} 0 ${-chassis_size_z/2.0+ground_gap_offset/2.0}" rpy="0 0 0"/>
-<parent link="chassis"/>
-<child link="front_chassis_caster"/>
-<axis xyz="0 1 0" rpy="0 0 0"/>
-<axis2 xyz="1 0 0" rpy="0 0 0"/>
-<limit effort="1000.0" lower="0.0" upper="3.14" velocity="0.5"/>
 </joint>
 <link name='left_wheel'>
+<pose xyz="0 0 0" rpy="0 0 0" />
         <inertial>
         <mass value="5.0"/>
@@ -161,5 +193,5 @@
         </inertial>
     <collision name='left_wheel_collision'>
-        <origin xyz="0 ${chassis_size_y/2.0 + wheel_length/2.0} 0" rpy="0 1.5707 1.5707"/>
+        <origin xyz="0 ${wheel_length/2} 0" rpy="0 1.5707 1.5707"/>
             <geometry>
             <cylinder radius="${wheel_radius}" length="${wheel_length}"/>
@@ -167,5 +199,5 @@
             </collision>
         <visual name='left_wheel_visual'>
-        <origin xyz="0 ${chassis_size_y/2.0 + wheel_length/2.0} 0" rpy=" 0 1.5707 1.5707"/>
+        <origin xyz="0 ${wheel_length/2} 0" rpy=" 0 1.5707 1.5707"/>
             <geometry>
             <cylinder radius="${wheel_radius}" length="${wheel_length}"/>
@@ -175,12 +207,11 @@
 </link>
 <joint name="left_wheel_hinge" type="continuous">
-<orgin xyz="0 ${chassis_size_y/2.0+0.1} 0" rpy="0 0 0"/>
+<origin xyz="0 ${chassis_size_y/2} 0" rpy="0 0 0"/>
 <parent link="chassis"/>
 <child link="left_wheel"/>
 <axis xyz="0 1 0" rpy="0 0 0"/>
-<limit effort="10000" velocity="1000"/>
-<dynamics damping="1.0" friction="0.01"/>
 </joint>
 <link name='right_wheel'>
+<pose xyz="0 0 0" rpy="0 0 0" />
         <inertial>
         <mass value="5.0"/>
@@ -191,5 +222,5 @@
         </inertial>
     <collision name='right_wheel_collision'>
-        <origin xyz="0 ${-(chassis_size_y/2.0 + wheel_length/2.0)} 0" rpy="0 1.5707 1.5707"/>
+        <origin xyz="0 ${-wheel_length/2} 0" rpy="0 1.5707 1.5707"/>
             <geometry>
             <cylinder radius="${wheel_radius}" length="${wheel_length}"/>
@@ -197,5 +228,5 @@
         </collision>
         <visual name='right_wheel_visual'>
-        <origin xyz="0 ${-(chassis_size_y/2.0 + wheel_length/2.0)} 0" rpy=" 0 1.5707 1.5707"/>
+        <origin xyz="0 ${-wheel_length/2} 0" rpy=" 0 1.5707 1.5707"/>
             <geometry>
             <cylinder radius="${wheel_radius}" length="${wheel_length}"/>
@@ -207,10 +238,8 @@
 </link>
 <joint name="right_wheel_hinge" type="continuous">
-<orgin xyz="0 ${-chassis_size_y/2.0-0.1} 0" rpy="0 0 0"/>
+<origin xyz="0 ${-chassis_size_y/2} 0" rpy="0 0 0"/>
 <parent link="chassis"/>
 <child link="right_wheel"/>
 <axis xyz="0 1 0" rpy="0 0 0"/>
-<limit effort="10000" velocity="1000"/>
-<dynamics damping="1.0" friction="0.01"/>
 </joint>
 <!---camera-->
@@ -278,6 +307,16 @@
 <dynamics damping="1.0" friction="1.0"/>
 </joint>
- <gazebo reference="camera">
+<gazebo reference="camera">
     <material>Gazebo/Green</material>
+  </gazebo>
+   <gazebo reference="back_wheel_chassis">
+    <mu1>0.2</mu1>
+    <mu2>0.2</mu2>
+    <material>Gazebo/Orange</material>
+  </gazebo>
+  <gazebo reference="front_wheel_chassis">
+      <mu1>0.2</mu1>
+    <mu2>0.2</mu2>
+    <material>Gazebo/Orange</material>
   </gazebo>
    <gazebo reference="left_wheel">
@@ -287,15 +326,12 @@
     <material>Gazebo/Red</material>
   </gazebo>
+  <gazebo reference="back_chassis_wheel">
+    <material>Gazebo/Red</material>
+  </gazebo>
+   <gazebo reference="front_chassis_wheel">
+    <material>Gazebo/Red</material>
+  </gazebo>
   <gazebo reference="chassis">
     <material>Gazebo/Orange</material>
   </gazebo>
-<gazebo reference="chassis_extra">
-    <material>Gazebo/Blue</material>
-  </gazebo>
-<gazebo reference="back_chassis_caster">
-    <material>Gazebo/OraBluenge</material>
-  </gazebo>
-<gazebo reference="front_chassis_caster">
-    <material>Gazebo/Blue</material>
-  </gazebo>
 </robot>
